File: FreqSynth.kicad_pcb (KiCad board)
At the start: 4 copper layers, 0 parts

Commit message: Fixed Amplifier, Added manf# field, ERC cleanup
Signed-off-by: Martin Berglund <LeastSignificantBit@users.noreply.github.com>
Other:
- rule pad_to_mask_clearance: 0.2 -> 0
Changed lines of the file:
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@@
 (kicad_pcb (version 20160815) (host pcbnew "(2016-08-28 BZR 7099, Git 440f8c8)-product")
   (general
-    (links 219)
-    (no_connects 100)
-    (area 56.794772 46.000144 172.025439 108.744144)
+    (links 0)
+    (no_connects 0)
+    (area 0 0 0 0)
     (thickness 1.6)
     (drawings 0)
@@
   )
   (layers
-    (0 F.Cu jumper)
-    (1 In1.Cu signal)
-    (2 In2.Cu signal)
+    (0 F.Cu signal)
+    (1 In1.Cu power)
+    (2 In2.Cu mixed)
     (31 B.Cu signal)
     (35 F.Paste user)
@@
     (pad_size 1.524 1.524)
     (pad_drill 0.762)
-    (pad_to_mask_clearance 0.2)
+    (pad_to_mask_clearance 0)
+    (pad_to_paste_clearance -0.1)
     (aux_axis_origin 0 0)
     (visible_elements FFFFFF7F)
@@
     (diff_pair_gap 0.25)
     (diff_pair_width 0.2)
-    (add_net /Amplifier/ATTEN_CS)
-    (add_net /Amplifier/RF_IN)
-    (add_net /Amplifier/RF_OUT)
-    (add_net /Clock/EXT_REF)
-    (add_net /Filter/FILT1)
-    (add_net /Filter/FILT2)
-    (add_net /Filter/FILT3)
-    (add_net /Filter/FILT4)
-    (add_net /Filter/VCC_RF)
-    (add_net /MCU/CE_PLL)
-    (add_net /MCU/CS_PLL)
-    (add_net /MCU/D+)
-    (add_net /MCU/D-)
-    (add_net /MCU/EN_PLL)
-    (add_net /MCU/EXT_CLK_EN)
-    (add_net /MCU/FILT1)
-    (add_net /MCU/FILT2)
-    (add_net /MCU/FILT3)
-    (add_net /MCU/FILT4)
-    (add_net /MCU/LD_PLL)
-    (add_net /MCU/SS_EXT)
-    (add_net /MISO)
-    (add_net /MOSI)
-    (add_net /PLL/CLK_REF)
-    (add_net /PLL/RF+)
-    (add_net /PLL/RF-)
-    (add_net /PLL/RFA_N)
-    (add_net /PLL/RFA_P)
-    (add_net /PLL/RFB_N)
-    (add_net /PLL/RFB_P)
-    (add_net /PLL/RF_BALANCED+)
-    (add_net /PLL/RF_BALANCED-)
-    (add_net /PLL/TUNE)
-    (add_net /PLL/VCC_PLL)
-    (add_net /Power/VIN)
-    (add_net /Power/VUSB)
-    (add_net /SCK)
-    (add_net Earth)
-    (add_net GNDD)
-    (add_net GNDPWR)
-    (add_net "Net-(C1-Pad2)")
-    (add_net "Net-(C18-Pad2)")
-    (add_net "Net-(C19-Pad2)")
-    (add_net "Net-(C2-Pad1)")
-    (add_net "Net-(C20-Pad2)")
-    (add_net "Net-(C25-Pad2)")
-    (add_net "Net-(C26-Pad2)")
-    (add_net "Net-(C27-Pad1)")
-    (add_net "Net-(C7-Pad1)")
-    (add_net "Net-(C7-Pad2)")
-    (add_net "Net-(D2-Pad2)")
-    (add_net "Net-(D3-Pad1)")
-    (add_net "Net-(D3-Pad2)")
-    (add_net "Net-(IC1-Pad18)")
-    (add_net "Net-(IC1-Pad19)")
-    (add_net "Net-(IC1-Pad20)")
-    (add_net "Net-(IC1-Pad21)")
-    (add_net "Net-(IC1-Pad24)")
-    (add_net "Net-(IC1-Pad25)")
-    (add_net "Net-(IC1-Pad5)")
-    (add_net "Net-(P2-Pad4)")
-    (add_net "Net-(P9-Pad2)")
-    (add_net "Net-(R1-Pad2)")
-    (add_net "Net-(R4-Pad2)")
-    (add_net "Net-(U5-Pad1)")
-    (add_net "Net-(U5-Pad10)")
-    (add_net "Net-(U5-Pad3)")
-    (add_net "Net-(U5-Pad5)")
-    (add_net "Net-(U5-Pad6)")
-    (add_net "Net-(U6-Pad3)")
-    (add_net "Net-(U7-Pad1)")
-    (add_net "Net-(U8-Pad1)")
-    (add_net "Net-(U8-Pad2)")
-    (add_net "Net-(U8-Pad3)")
-    (add_net "Net-(U8-Pad4)")
-    (add_net "Net-(U8-Pad5)")
-    (add_net "Net-(U8-Pad6)")
-    (add_net "Net-(U8-Pad7)")
-    (add_net "Net-(U8-Pad8)")
-    (add_net "Net-(U8-Pad9)")
-    (add_net VCC)
   )
 )

Commit message: Started on the board even though theres some components missing
Signed-off-by: Martin Berglund <LeastSignificantBit@users.noreply.github.com>
Parts:
- added C1: 10nF, Capacitors_SMD:C_0603, F.Cu at (88.3, 114.2)
- added C10: 1nF_RF, Capacitors_SMD:C_0402, F.Cu at (106.4, 106.4)
- added C11: 10nF, Capacitors_SMD:C_0603, F.Cu at (113.6, 109.0)
- added C12: 1nF_RF, Capacitors_SMD:C_0402, F.Cu at (119.3, 91.7)
- added C13: 10nF, Capacitors_SMD:C_0603, F.Cu at (122.5, 97.6)
- added C14: 100pF, Capacitors_SMD:C_0603, F.Cu at (117.9, 97.6)
- added C15: 10nF, Capacitors_SMD:C_0603, F.Cu at (116.3, 102.9)
- added C16: 100pF, Capacitors_SMD:C_0603, F.Cu at (121.1, 91.9)
- added C17: 10nF, Capacitors_SMD:C_0603, F.Cu at (119.1, 109.0)
- added C18: 100pF, Capacitors_SMD:C_0603, F.Cu at (109.0, 103.3)
- added C19: 10nF, Capacitors_SMD:C_0603, F.Cu at (113.4, 97.6)
- added C2: 1uF, Capacitors_SMD:C_0603, F.Cu at (121.7, 103.3)
- added C20: 100pF, Capacitors_SMD:C_0603, F.Cu at (116.5, 108.6)
- added C21: 10nF, Capacitors_SMD:C_0603, F.Cu at (109.3, 97.6)
- added C22: 100pF, Capacitors_SMD:C_0603, F.Cu at (111.8, 102.9)
- added C23: 10nF, Capacitors_SMD:C_0603, F.Cu at (117.7, 97.2)
- added C24: 100pF, Capacitors_SMD:C_0603, F.Cu at (113.2, 97.2)
- added C25: 1nF_RF, Capacitors_SMD:C_0402, F.Cu at (113.6, 91.7)
- added C26: 10nF, Capacitors_SMD:C_0603, F.Cu at (94.2, 115.4)
- added C27: 100pF, Capacitors_SMD:C_0603, F.Cu at (94.2, 116.7)
- added C28: 1µF, Capacitors_SMD:C_0603, F.Cu at (56.6, 74.8)
- added C29: 100nF, Capacitors_SMD:C_0603, F.Cu at (67.4, 70.5)
- added C3: 1uF, Capacitors_SMD:C_0603, F.Cu at (126.4, 103.2)
- added C30: 10µF, Capacitors_SMD:C_0805, F.Cu at (61.1, 72.1)
- added C31: 1µF, Capacitors_SMD:C_0603, F.Cu at (63.2, 74.4)
- added C32: 1µF, Capacitors_SMD:C_0603, F.Cu at (59.9, 74.8)
- added C33: 100nF, Capacitors_SMD:C_0603, F.Cu at (68.0, 71.9)
- added C34: 10µF, Capacitors_SMD:C_0805, F.Cu at (56.9, 72.1)
- added C35: 1µF, Capacitors_SMD:C_0603, F.Cu at (66.5, 76.2)
- added C36: 1µF, Capacitors_SMD:C_0603, F.Cu at (71.6, 71.8)
- added C37: 100nF, Capacitors_SMD:C_0603, F.Cu at (67.8, 66.4)
- added C38: 10nF, Capacitors_SMD:C_0603, F.Cu at (63.4, 71.9)
- added C39: 100pF_RF, Capacitors_SMD:C_0402, F.Cu at (102.2, 68.0)
- added C4: 1uF, Capacitors_SMD:C_0603, F.Cu at (122.2, 97.6)
- added C40: 100pF_RF, Capacitors_SMD:C_0402, F.Cu at (107.2, 68.0)
- added C41: 6pF_RF, Capacitors_SMD:C_0402, F.Cu at (104.7, 68.8)
- added C42: 0.5pF_RF, Capacitors_SMD:C_0402, F.Cu at (102.9, 70.8)
- added C43: 0.5pF_RF, Capacitors_SMD:C_0402, F.Cu at (107.4, 70.8)
- added C44: 2pF_RF, Capacitors_SMD:C_0402, F.Cu at (105.2, 71.5)
- added C45: 0.8pF_RF, Capacitors_SMD:C_0402, F.Cu at (102.4, 73.5)
- added C46: 0.8pF_RF, Capacitors_SMD:C_0402, F.Cu at (106.9, 73.5)
- added C47: 4pF_RF, Capacitors_SMD:C_0402, F.Cu at (104.7, 74.3)
- added C48: 2.4pF_RF, Capacitors_SMD:C_0402, F.Cu at (102.9, 76.3)
- added C49: 2.4pF_RF, Capacitors_SMD:C_0402, F.Cu at (107.4, 76.3)
- added C5: 100nF, Capacitors_SMD:C_0603, F.Cu at (109.0, 109.0)
- added C50: 5pF_RF, Capacitors_SMD:C_0402, F.Cu at (105.2, 75.5)
- added C51: 1µF, Capacitors_SMD:C_0603, F.Cu at (125.7, 69.5)
- added C52: 10nF, Capacitors_SMD:C_0603, F.Cu at (127.7, 68.8)
- added C53: 100nF, Capacitors_SMD:C_0603, F.Cu at (125.7, 71.0)
- added C54: 10pF, Capacitors_SMD:C_0603, F.Cu at (127.7, 70.3)
- added C55: 1nF_RF, Capacitors_SMD:C_0402, F.Cu at (117.1, 72.5)
- added C56: 1nF_RF, Capacitors_SMD:C_0402, F.Cu at (124.2, 72.5)
- added C57: 1nF_RF, Capacitors_SMD:C_0402, F.Cu at (132.2, 72.5)
- added C58: 1nF_RF, Capacitors_SMD:C_0402, F.Cu at (130.2, 75.0)
- added C59: 10nF, Capacitors_SMD:C_0603, F.Cu at (117.7, 70.3)
- added C6: 10nF, Capacitors_SMD:C_0603, F.Cu at (126.5, 97.6)
- added C60: 100pF, Capacitors_SMD:C_0603, F.Cu at (116.7, 70.3)
- added C61: 22p, Capacitors_SMD:C_0402, F.Cu at (80.3, 87.1)
- added C62: 22p, Capacitors_SMD:C_0402, F.Cu at (80.3, 86.3)
- added C63: 1µF, Capacitors_SMD:C_0603, F.Cu at (73.6, 90.8)
- added C7: 12nF, Capacitors_SMD:C_0603, F.Cu at (122.4, 91.9)
- added C8: 820pF, Capacitors_SMD:C_0603, F.Cu at (118.8, 103.3)
- added C9: 1nF_RF, Capacitors_SMD:C_0402, F.Cu at (106.4, 101.1)
- added D1: CPL-DIO-MBR0520, Diodes_SMD:SOD-123, F.Cu at (69.1, 63.3)
- added D2: CPL-LED-0603-GREEN, LEDs:LED_0603, F.Cu at (56.3, 68.4)
- added D3: CPL-LED-0603-YELLOW, LEDs:LED_0603, F.Cu at (81.4, 93.3)
- added IC1: ATMEGA32U2, Housings_QFP:TQFP-32_7x7mm_Pitch0.8mm, F.Cu at (74.3, 84.3)
- added L1: 8nH, FreqSynth:L_0402, F.Cu at (103.7, 68.0)
- added L10: 6.1nH, FreqSynth:L_0402, F.Cu at (104.4, 76.3)
- added L11: 6.1nH, FreqSynth:L_0402, F.Cu at (105.9, 76.3)
- added L12: 3nH, FreqSynth:L_0402, F.Cu at (105.2, 77.0)
- added L13: 100nH, FreqSynth:L_0603, F.Cu at (128.4, 71.8)
- added L2: 8nH, FreqSynth:L_0402, F.Cu at (105.7, 68.0)
- added L3: 200nH, FreqSynth:L_0603, F.Cu at (104.7, 67.0)
- added L4: 2.5nH, FreqSynth:L_0402, F.Cu at (104.4, 70.8)
- added L5: 2.5nH, FreqSynth:L_0402, F.Cu at (105.9, 70.8)
- added L6: 0.6nH, FreqSynth:L_0402, F.Cu at (105.2, 70.0)
- added L7: 5nH, FreqSynth:L_0402, F.Cu at (103.9, 73.5)
- added L8: 5nH, FreqSynth:L_0402, F.Cu at (105.4, 73.5)
- added L9: 1nH, FreqSynth:L_0402, F.Cu at (104.7, 72.8)
- added P1: CPL-CON-BARREL-2.1MM, Connect:BARREL_JACK, F.Cu at (43.5, 65.0)
- added P10: RESET, Pin_Headers:Pin_Header_Straight_1x01, F.Cu at (69.3, 93.3)
- added P2: RF1, FreqSynth:SMA_edge, F.Cu at (137.2, 72.5)
- added P3: RF2P, FreqSynth:SMA_edge, F.Cu at (137.2, 97.2)
- added P4: RF2N, FreqSynth:SMA_edge, F.Cu at (137.2, 111.0)
- added P5: 61729-1011BLF, FreqSynth:FCI_61729-1011BLF, F.Cu at (47.0, 81.0)
- added P6: CONN_01X06, Pin_Headers:Pin_Header_Angled_1x06, F.Cu at (49.8, 105.2)
- added P7: REF_IN, FreqSynth:SMA_edge, F.Cu at (42.5, 114.5)
- added P8: VTEST, Pin_Headers:Pin_Header_Straight_1x03, F.Cu at (75.1, 64.6)
- added P9: PWRSEL, Pin_Headers:Pin_Header_Straight_1x03, F.Cu at (63.9, 63.2)
- added R1: 5.1k, Resistors_SMD:R_0603, F.Cu at (123.1, 103.3)
- added R10: 0R, Resistors_SMD:R_0603, F.Cu at (69.4, 74.4)
- added R11: 33R, Resistors_SMD:R_0603, F.Cu at (72.0, 66.4)
- added R12: 49.9R, Resistors_SMD:R_0603, F.Cu at (99.4, 75.3)
- added R13: 1.8R, Resistors_SMD:R_0603, F.Cu at (127.7, 67.3)
- added R14: 100R, Resistors_SMD:R_0402, F.Cu at (130.2, 73.3)
- added R15: 10k, Resistors_SMD:R_0603, F.Cu at (69.6, 88.8)
- added R16: 1M, Resistors_SMD:R_0603, F.Cu at (81.9, 86.7)
- added R17: 33R, Resistors_SMD:R_0603, F.Cu at (78.7, 92.5)
- added R2: 30.1R, Resistors_SMD:R_0603, F.Cu at (118.0, 109.0)
- added R3: 49.9R, Resistors_SMD:R_0603, F.Cu at (122.7, 109.0)
- added R4: 49.9R, Resistors_SMD:R_0603, F.Cu at (126.0, 91.9)
- added R5: 90.9R, Resistors_SMD:R_0603, F.Cu at (113.9, 103.3)
- added R6: 240R, Resistors_SMD:R_0603, F.Cu at (111.8, 91.9)
- added R7: 49.9R, Resistors_SMD:R_0603, F.Cu at (116.3, 91.9)
- added R8: 49.9R, Resistors_SMD:R_0603, F.Cu at (111.6, 108.6)
- added R9: 0R, Resistors_SMD:R_0603, F.Cu at (66.3, 74.4)
- added RESET1: B3F-1000, FreqSynth:SW_B3F-1000, F.Cu at (62.3, 86.8)
- added U1: MAX2870, Housings_DFN_QFN:QFN-32-1EP_5x5mm_Pitch0.5mm, F.Cu at (107.1, 93.8)
- added U2: TS5A3159, TO_SOT_Packages_SMD:SC-70-6, F.Cu at (94.2, 113.4)
- added U5: CPL-REG-LIN-3.3V-0.15A, TO_SOT_Packages_SMD:SOT-23-5, F.Cu at (58.3, 65.5)
- added U6: SKY13322-375LF, FreqSynth:MLPD-10, F.Cu at (109.8, 72.3)
- added U7: SKY13322-375LF, FreqSynth:MLPD-10, F.Cu at (100.3, 72.3)
- added U8: TRF37A75, Housings_DFN_QFN:DFN-8-1EP_2x2mm_Pitch0.5mm, F.Cu at (126.5, 72.8)
- added U9: PE43711, Housings_DFN_QFN:QFN-24-1EP_4x4mm_Pitch0.5mm, F.Cu at (120.7, 71.8)
- added X1: 25MHz ±5ppm 3.3V 33mA, Crystals:Crystal_SMD_2520_4Pads, F.Cu at (94.2, 109.6)
- added X2: 8MHz 18PF 50ppm, Crystals:Crystal_SMD_5032_4Pads, F.Cu at (84.7, 86.7)
Other:
- board outline added: 100 x 60 mm

Commit message: Added a todolist and solved som small crap
Signed-off-by: Martin Berglund <LeastSignificantBit@users.noreply.github.com>
Parts:
- moved P3 14.9 mm to (136.0, 112.0)
- moved P4 14.0 mm to (137.0, 97.0)
- moved P7 4.53 mm to (47.0, 114.0), turned to 180 degrees
- moved P2 0.20 mm to (137.0, 72.7)
Other:
- outline, holes or cut-outs redrawn

Commit message: Outline starts to come togeter
Signed-off-by: Martin Berglund <LeastSignificantBit@users.noreply.github.com>
Parts:
- added R?: 0R, Resistors_SMD:R_0603, F.Cu at (57.4, 138.2)
- moved C9 108.9 mm to (206.8, 143.4)
- moved C10 103.3 mm to (202.8, 143.6)
- moved C19 101.1 mm to (202.2, 146.0)
- moved C21 101.1 mm to (198.1, 146.0)
- moved C24 101.1 mm to (202.0, 145.6)
- moved U1 101.1 mm to (195.9, 142.2)
- moved C14 101.1 mm to (206.7, 146.0)
- moved C23 101.1 mm to (206.5, 145.6)
- moved C25 101.1 mm to (202.4, 140.1)
- moved C15 101.1 mm to (205.1, 151.3)
- moved R6 101.1 mm to (200.6, 140.3)
- moved C18 101.1 mm to (197.8, 151.7)
- moved C2 101.1 mm to (210.5, 151.7)
- moved C22 101.1 mm to (200.6, 151.3)
- moved C8 101.1 mm to (207.6, 151.7)
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Connections:
- P6 pad 1: GNDPWR -> Net-(P6-Pad1)
- P6 pad 2: /Power/VIN -> Net-(P6-Pad2)
- P6 pad 3: /SCK -> Net-(P6-Pad3)
- P6 pad 4: /MOSI -> Net-(P6-Pad4)
- P6 pad 5: /MISO -> Net-(P6-Pad5)
Other:
- board size 100 x 60 mm -> 79 x 50 mm

Commit message: Fixed USB mini B
Signed-off-by: Martin Berglund <LeastSignificantBit@users.noreply.github.com>
Parts:
- removed R?: 0R, Resistors_SMD:R_0603
- added R18: 0R, Resistors_SMD:R_0603, F.Cu at (56.0, 138.6)
- P5: value 61729-1011BLF -> USB_MINI_B; footprint FreqSynth:FCI_61729-1011BLF -> FreqSynth:conn_usb_B_mini_smd
- moved P1 16.0 mm to (105.8, 108.8)
- moved P5 11.4 mm to (103.4, 121.8), turned to 270 degrees
Connections:
- P5 pad 4: GNDPWR -> Net-(P5-Pad4)
Changed lines of the file:
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@@
 (kicad_pcb (version 20160815) (host pcbnew 4.X.X-head)
   (general
-    (links 296)
-    (no_connects 281)
+    (links 298)
+    (no_connects 283)
     (area 100.424999 99.924999 179.575001 150.075001)
     (thickness 1.6)
@@
     (zones 0)
     (modules 118)
-    (nets 98)
+    (nets 99)
   )
   (page A4)
@@
   (net 96 "Net-(P6-Pad4)")
   (net 97 "Net-(P6-Pad5)")
+  (net 98 "Net-(P5-Pad4)")
   (net_class Default "This is the default net class."
     (clearance 0.127)
@@
     (add_net "Net-(IC1-Pad25)")
     (add_net "Net-(IC1-Pad5)")
+    (add_net "Net-(P5-Pad4)")
     (add_net "Net-(P6-Pad1)")
     (add_net "Net-(P6-Pad2)")
@@
     )
   )
-  (module FreqSynth:FCI_61729-1011BLF (layer F.Cu)
-    (at 108.8 111.8 90)
-    (solder_mask_margin 0.1)
-    (fp_text reference P5 (at -5.79 -11.635 90) (layer F.SilkS)
-      (effects (font (size 0.4 0.4) (thickness 0.1)))
-    )
-    (fp_text value 61729-1011BLF (at -5.075 7.615 90) (layer F.SilkS)
-      (effects (font (size 0.4 0.4) (thickness 0.1)))
-    )
-    (fp_line (start 6 -2) (end 6 -10.5) (layer F.SilkS) (width 0.127))
-    (fp_line (start -6 -2) (end -6 -10.5) (layer F.SilkS) (width 0.127))
-    (fp_line (start 6 -10.5) (end -6 -10.5) (layer F.SilkS) (width 0.127))
-    (fp_line (start 6 5.5) (end -6 5.5) (layer F.SilkS) (width 0.127))
-    (fp_line (start 6 5.5) (end 6 2) (layer F.SilkS) (width 0.127))
-    (fp_line (start -6 5.5) (end -6 2) (layer F.SilkS) (width 0.127))
-    (fp_circle (center -2.98 6.4) (end -2.726 6.4) (layer F.SilkS) (width 0))
-    (fp_line (start -8 6) (end 8 6) (layer Dwgs.User) (width 0.127))
-    (fp_line (start 8 6) (end 8 -10.75) (layer Dwgs.User) (width 0.127))
-    (fp_line (start 8 -10.75) (end -8 -10.75) (layer Dwgs.User) (width 0.127))
-    (fp_line (start -8 -10.75) (end -8 6) (layer Dwgs.User) (width 0.127))
-    (pad 1 thru_hole circle (at -1.25 4.71 270) (size 1.508 1.508) (drill 1) (layers *.Cu *.Mask F.SilkS)
-      (net 32 /Power/VUSB) (solder_mask_margin 0.2))
-    (pad 2 thru_hole circle (at 1.25 4.71 270) (size 1.508 1.508) (drill 1) (layers *.Cu *.Mask F.SilkS)
-      (net 55 /MCU/D-) (solder_mask_margin 0.2))
-    (pad 3 thru_hole circle (at 1.25 2.71 270) (size 1.508 1.508) (drill 1) (layers *.Cu *.Mask F.SilkS)
-      (net 54 /MCU/D+) (solder_mask_margin 0.2))
-    (pad 4 thru_hole circle (at -1.25 2.71 270) (size 1.508 1.508) (drill 1) (layers *.Cu *.Mask F.SilkS)
-      (net 24 GNDPWR) (solder_mask_margin 0.2))
-    (pad S1 thru_hole circle (at -6.02 0 270) (size 3.416 3.416) (drill 2.4) (layers *.Cu *.Mask F.SilkS)
-      (net 24 GNDPWR) (solder_mask_margin 0.2))
-    (pad S2 thru_hole circle (at 6.02 0 270) (size 3.416 3.416) (drill 2.4) (layers *.Cu *.Mask F.SilkS)
-      (net 24 GNDPWR) (solder_mask_margin 0.2))
-    (model ${KISYS3DMOD}/Connect.3dshapes/USB_B.wrl
-      (at (xyz 0 0 0))
-      (scale (xyz 0.4 0.4 0.4))
-      (rotate (xyz 0 0 180))
-    )
-  )
   (module Diodes_SMD:SOD-123 (layer F.Cu)
     (at 136.9 84.1)
@@
   )
   (module Connect:BARREL_JACK (layer F.Cu)
-    (at 105.59934 124.8)
+    (at 105.79986 108.8)
     (descr "DC Barrel Jack")
     (tags "Power Jack")
@@
     )
   )
-  (module Resistors_SMD:R_0603 (layer F.Cu)
-    (at 57.4 138.2)
-    (descr "Resistor SMD 0603, reflow soldering, Vishay (see dcrcw.pdf)")
-    (tags "resistor 0603")
-    (attr smd)
-    (fp_text reference R? (at 0 -1.9) (layer F.SilkS)
-      (effects (font (size 1 1) (thickness 0.15)))
-    )
-    (fp_text value 0R (at 0 1.9) (layer F.Fab)
-      (effects (font (size 1 1) (thickness 0.15)))
-    )
-    (fp_line (start -1.3 -0.8) (end 1.3 -0.8) (layer F.CrtYd) (width 0.05))
-    (fp_line (start -1.3 0.8) (end 1.3 0.8) (layer F.CrtYd) (width 0.05))
-    (fp_line (start -1.3 -0.8) (end -1.3 0.8) (layer F.CrtYd) (width 0.05))
-    (fp_line (start 1.3 -0.8) (end 1.3 0.8) (layer F.CrtYd) (width 0.05))
-    (fp_line (start 0.5 0.675) (end -0.5 0.675) (layer F.SilkS) (width 0.15))
-    (fp_line (start -0.5 -0.675) (end 0.5 -0.675) (layer F.SilkS) (width 0.15))
-    (pad 1 smd rect (at -0.75 0) (size 0.5 0.9) (layers F.Cu F.Paste F.Mask)
-      (net 93 "Net-(P6-Pad1)"))
-    (pad 2 smd rect (at 0.75 0) (size 0.5 0.9) (layers F.Cu F.Paste F.Mask)
-      (net 24 GNDPWR))
-    (model Resistors_SMD.3dshapes/R_0603.wrl
-      (at (xyz 0 0 0))
-      (scale (xyz 1 1 1))
-      (rotate (xyz 0 0 0))
-    )
-  )
   (module FreqSynth:SMA_edge (layer F.Cu)
     (at 104.8 142.9 180)
@@
     )
   )
+  (module Resistors_SMD:R_0603 (layer F.Cu)
+    (at 56.05 138.6)
+    (descr "Resistor SMD 0603, reflow soldering, Vishay (see dcrcw.pdf)")
+    (tags "resistor 0603")
+    (attr smd)
+    (fp_text reference R18 (at 0 -1.9) (layer F.SilkS)
+      (effects (font (size 1 1) (thickness 0.15)))
+    )
+    (fp_text value 0R (at 0 1.9) (layer F.Fab)
+      (effects (font (size 1 1) (thickness 0.15)))
+    )
+    (fp_line (start -1.3 -0.8) (end 1.3 -0.8) (layer F.CrtYd) (width 0.05))
+    (fp_line (start -1.3 0.8) (end 1.3 0.8) (layer F.CrtYd) (width 0.05))
+    (fp_line (start -1.3 -0.8) (end -1.3 0.8) (layer F.CrtYd) (width 0.05))
+    (fp_line (start 1.3 -0.8) (end 1.3 0.8) (layer F.CrtYd) (width 0.05))
+    (fp_line (start 0.5 0.675) (end -0.5 0.675) (layer F.SilkS) (width 0.15))
+    (fp_line (start -0.5 -0.675) (end 0.5 -0.675) (layer F.SilkS) (width 0.15))
+    (pad 1 smd rect (at -0.75 0) (size 0.5 0.9) (layers F.Cu F.Paste F.Mask)
+      (net 93 "Net-(P6-Pad1)"))
+    (pad 2 smd rect (at 0.75 0) (size 0.5 0.9) (layers F.Cu F.Paste F.Mask)
+      (net 24 GNDPWR))
+    (model Resistors_SMD.3dshapes/R_0603.wrl
+      (at (xyz 0 0 0))
+      (scale (xyz 1 1 1))
+      (rotate (xyz 0 0 0))
+    )
+  )
+  (module FreqSynth:conn_usb_B_mini_smd (layer F.Cu)
+    (at 103.4 121.8 270)
+    (descr "USB B mini SMD connector")
+    (fp_text reference P5 (at 0 6.10108 270) (layer F.SilkS)
+      (effects (font (size 0.99822 0.99822) (thickness 0.19558)))
+    )
+    (fp_text value USB_MINI_B (at 0 -5.90042 270) (layer F.SilkS)
+      (effects (font (size 0.99822 0.99822) (thickness 0.19812)))
+    )
+    (fp_line (start -3.8989 -4.40436) (end -5.00126 -4.40436) (layer F.SilkS) (width 0.3048))
+    (fp_line (start -5.00126 -4.40436) (end -5.00126 -2.90322) (layer F.SilkS) (width 0.3048))
+    (fp_line (start -5.00126 -2.90322) (end -3.8989 -2.90322) (layer F.SilkS) (width 0.3048))
+    (fp_line (start 5.00126 -2.90068) (end 3.8989 -2.90068) (layer F.SilkS) (width 0.3048))
+    (fp_line (start 5.00126 -4.40182) (end 5.00126 -2.90068) (layer F.SilkS) (width 0.3048))
+    (fp_line (start 3.8989 -4.40182) (end 5.00126 -4.40182) (layer F.SilkS) (width 0.3048))
+    (fp_line (start 3.8989 1.09982) (end 5.00126 1.09982) (layer F.SilkS) (width 0.3048))
+    (fp_line (start 5.00126 1.09982) (end 5.00126 2.60096) (layer F.SilkS) (width 0.3048))
+    (fp_line (start 5.00126 2.60096) (end 3.8989 2.60096) (layer F.SilkS) (width 0.3048))
+    (fp_line (start -3.8989 1.09982) (end -5.00126 1.09982) (layer F.SilkS) (width 0.3048))
+    (fp_line (start -5.00126 1.09982) (end -5.00126 2.60096) (layer F.SilkS) (width 0.3048))
+    (fp_line (start -5.00126 2.60096) (end -3.8989 2.60096) (layer F.SilkS) (width 0.3048))
+    (fp_line (start -3.8989 5.00126) (end 3.8989 5.00126) (layer F.SilkS) (width 0.3048))
+    (fp_line (start 3.8989 5.00126) (end 3.8989 -5.00126) (layer F.SilkS) (width 0.3048))
+    (fp_line (start 3.8989 -5.00126) (end -3.8989 -5.00126) (layer F.SilkS) (width 0.3048))
+    (fp_line (start -3.8989 -5.00126) (end -3.8989 5.00126) (layer F.SilkS) (width 0.3048))
+    (pad 6 smd rect (at 4.42976 -3.6195 270) (size 2.1971 2.1971) (layers F.Cu F.Paste F.Mask)
+      (net 24 GNDPWR))
+    (pad 1 smd rect (at -1.59766 -3.8989 270) (size 0.49784 2.1971) (layers F.Cu F.Paste F.Mask)
+      (net 32 /Power/VUSB))
+    (pad 2 smd rect (at -0.79756 -3.8989 270) (size 0.49784 2.1971) (layers F.Cu F.Paste F.Mask)
+      (net 55 /MCU/D-))
+    (pad 3 smd rect (at 0 -3.8989 270) (size 0.49784 2.1971) (layers F.Cu F.Paste F.Mask)
+      (net 54 /MCU/D+))
+    (pad 4 smd rect (at 0.79756 -3.8989 270) (size 0.49784 2.1971) (layers F.Cu F.Paste F.Mask)
+      (net 98 "Net-(P5-Pad4)"))
+    (pad 5 smd rect (at 1.59766 -3.8989 270) (size 0.49784 2.1971) (layers F.Cu F.Paste F.Mask)
+      (net 24 GNDPWR))
+    (pad "" np_thru_hole circle (at -2.1971 -1.3716 270) (size 0.89916 0.89916) (drill 0.89916) (layers *.Cu *.Mask F.SilkS))
+    (pad "" np_thru_hole circle (at 2.19964 -1.3716 270) (size 0.89916 0.89916) (drill 0.89916) (layers *.Cu *.Mask F.SilkS))
+    (pad 6 smd rect (at -4.42976 -3.6195 270) (size 2.1971 2.1971) (layers F.Cu F.Paste F.Mask)
+      (net 24 GNDPWR))
+    (pad 6 smd rect (at -4.42976 1.8796 270) (size 2.1971 2.1971) (layers F.Cu F.Paste F.Mask)
+      (net 24 GNDPWR))
+    (pad 6 smd rect (at 4.42976 1.8796 270) (size 2.1971 2.1971) (layers F.Cu F.Paste F.Mask)
+      (net 24 GNDPWR))
+    (model lib/usb_B_mini_smd.wrl
+      (at (xyz 0 0 0))
+      (scale (xyz 1 1 1))
+      (rotate (xyz 0 0 0))
+    )
+  )
