File: FreqSynth.kicad_pcb (KiCad board)
At the start: 4 copper layers, 49 x 50 mm, 411 parts, among them P1 CPL-CON-BARREL-2.1MM, P2 RF1, P3 RF2, P4 CONN_01X03, P5 REF_IN, P6 SWD, U1 MAX2870, U10 PE43711, U11 LMH2110, U12 STM32F030K6T6, U2 TS5A3159, U3 TLV7113333DDSET, U4 AP65101, U5 TLV7113333DDSET, U6 RT9069-50GB, U7 SKY13322-375LF, U8 SKY13322-375LF, U9 TRF37A75, X1 25MHz ±5ppm 3.3V 33mA

Commit message: Almost finished, Via stitching in place plus decals
Signed-off-by: Martin Berglund <LeastSignificantBit@users.noreply.github.com>
Parts:
- removed the ? at (148.0, 135.4)
- removed the ? at (147.0, 116.6)
- removed the ? at (143.0, 116.6)
- removed the ? at (143.0, 114.6)
- removed the ? at (145.0, 116.6)
- removed the ? at (145.0, 114.6)
- removed the ? at (147.0, 114.6)
- removed the ? at (145.0, 112.6)
- removed the ? at (147.0, 112.6)
- removed the ? at (148.0, 131.4)
- removed the ? at (165.2, 137.0)
- removed the ? at (161.2, 133.0)
- removed the ? at (167.2, 139.0)
- removed the ? at (164.2, 136.0)
- removed the ? at (166.2, 138.0)
- removed the ? at (162.2, 134.0)
- removed the ? at (163.2, 135.0)
- removed the ? at (168.2, 140.0)
- removed the ? at (155.8, 137.0)
- removed the ? at (159.8, 133.0)
- removed the ? at (153.8, 139.0)
- removed the ? at (156.8, 136.0)
- removed the ? at (154.8, 138.0)
- removed the ? at (158.8, 134.0)
- removed the ? at (157.8, 135.0)
- removed the ? at (152.8, 140.0)
- removed the ? at (158.8, 128.8)
- removed the ? at (159.8, 128.8)
- removed the ? at (159.8, 129.8)
- removed the ? at (158.8, 129.8)
- removed the ? at (156.8, 130.8)
- removed the ? at (157.8, 130.8)
- removed the ? at (155.8, 130.8)
- removed the ? at (157.8, 128.8)
- removed the ? at (155.8, 128.8)
- removed the ? at (156.8, 128.8)
- removed the ? at (156.8, 129.8)
- removed the ? at (157.8, 129.8)
- removed the ? at (152.8, 130.8)
- removed the ? at (153.8, 130.8)
- removed the ? at (153.8, 128.8)
- removed the ? at (152.8, 129.8)
- removed the ? at (154.8, 128.8)
- removed the ? at (154.8, 130.8)
- removed the ? at (152.8, 128.8)
- removed the ? at (153.8, 129.8)
- removed the ? at (157.8, 131.8)
- removed the ? at (158.8, 131.8)
- removed the ? at (158.8, 130.8)
- removed the ? at (159.8, 130.8)
- removed the ? at (159.8, 131.8)
- removed the ? at (156.8, 131.8)
- removed the ? at (152.8, 131.8)
- removed the ? at (154.8, 129.8)
- removed the ? at (154.8, 131.8)
- removed the ? at (155.8, 131.8)
- removed the ? at (155.8, 129.8)
- removed the ? at (153.8, 131.8)
- removed the ? at (157.8, 127.8)
- removed the ? at (156.8, 126.8)
- removed the ? at (159.8, 127.8)
- removed the ? at (158.8, 126.8)
- removed the ? at (159.8, 126.8)
- removed the ? at (156.8, 127.8)
- removed the ? at (157.8, 126.8)
- removed the ? at (158.8, 127.8)
- removed the ? at (154.8, 127.8)
- removed the ? at (155.8, 126.8)
- removed the ? at (153.8, 127.8)
- removed the ? at (155.8, 127.8)
- removed the ? at (152.8, 127.8)
- removed the ? at (158.8, 124.8)
- removed the ? at (159.8, 125.8)
- removed the ? at (159.8, 124.8)
- removed the ? at (156.8, 124.8)
- removed the ? at (156.8, 125.8)
- removed the ? at (158.8, 125.8)
- removed the ? at (157.8, 124.8)
- removed the ? at (157.8, 125.8)
- removed the ? at (155.8, 125.8)
- removed the ? at (148.0, 133.4)
- removed the ? at (146.0, 131.4)
- removed the ? at (146.0, 133.4)
- removed the ? at (146.0, 135.4)
- removed the ? at (144.0, 131.4)
- removed the ? at (144.0, 135.4)
- removed the ? at (143.0, 112.6)
- added ?: , FreqSynth:VIA, F.Cu at (142.4, 130.8)
- added ?: , FreqSynth:VIA, F.Cu at (116.8, 140.8)
- added ?: , FreqSynth:VIA, F.Cu at (127.2, 118.2)
- added ?: , FreqSynth:VIA, F.Cu at (121.4, 119.6)
- added ?: , FreqSynth:VIA, F.Cu at (122.4, 118.6)
- added ?: , FreqSynth:VIA, F.Cu at (123.4, 117.6)
- added ?: , FreqSynth:VIA, F.Cu at (107.2, 126.4)
- added ?: , FreqSynth:VIA, F.Cu at (108.2, 123.4)
- added ?: , FreqSynth:VIA, F.Cu at (109.2, 124.4)
- added ?: , FreqSynth:VIA, F.Cu at (107.2, 124.4)
- added ?: , FreqSynth:VIA, F.Cu at (106.2, 123.4)
- added ?: , FreqSynth:VIA, F.Cu at (119.8, 101.8)
- added ?: , FreqSynth:VIA, F.Cu at (117.8, 141.8)
- added ?: , FreqSynth:VIA, F.Cu at (121.8, 101.8)
- added ?: , FreqSynth:VIA, F.Cu at (122.8, 102.8)
- added ?: , FreqSynth:VIA, F.Cu at (120.8, 102.8)
- added ?: , FreqSynth:VIA, F.Cu at (121.8, 103.8)
- added ?: , FreqSynth:VIA, F.Cu at (119.8, 103.8)
- added ?: , FreqSynth:VIA, F.Cu at (146.4, 102.0)
- added ?: , FreqSynth:VIA, F.Cu at (144.4, 102.0)
- added ?: , FreqSynth:VIA, F.Cu at (142.4, 102.0)
- added ?: , FreqSynth:VIA, F.Cu at (135.4, 113.4)
- added ?: , FreqSynth:VIA, F.Cu at (136.6, 114.4)
- added ?: , FreqSynth:VIA, F.Cu at (122.8, 147.6)
- added ?: , FreqSynth:VIA, F.Cu at (136.6, 112.8)
- added ?: , FreqSynth:VIA, F.Cu at (136.6, 110.6)
- added ?: , FreqSynth:VIA, F.Cu at (137.8, 109.6)
- added ?: , FreqSynth:VIA, F.Cu at (139.6, 105.2)
- added ?: , FreqSynth:VIA, F.Cu at (140.6, 104.2)
- added ?: , FreqSynth:VIA, F.Cu at (138.6, 104.2)
- added ?: , FreqSynth:VIA, F.Cu at (141.6, 105.2)
- added ?: , FreqSynth:VIA, F.Cu at (129.0, 107.2)
- added ?: , FreqSynth:VIA, F.Cu at (127.5, 108.6)
- added ?: , FreqSynth:VIA, F.Cu at (127.5, 106.8)
- added ?: , FreqSynth:VIA, F.Cu at (121.8, 146.6)
- added ?: , FreqSynth:VIA, F.Cu at (126.5, 109.6)
- added ?: , FreqSynth:VIA, F.Cu at (126.5, 107.6)
- added ?: , FreqSynth:VIA, F.Cu at (131.3, 105.4)
- added ?: , FreqSynth:VIA, F.Cu at (133.3, 105.4)
- added ?: , FreqSynth:VIA, F.Cu at (132.3, 106.4)
- added ?: , FreqSynth:VIA, F.Cu at (130.3, 106.4)
- added ?: , FreqSynth:VIA, F.Cu at (129.3, 105.4)
- added ?: , FreqSynth:VIA, F.Cu at (122.8, 130.6)
- added ?: , FreqSynth:VIA, F.Cu at (121.8, 129.6)
- added ?: , FreqSynth:VIA, F.Cu at (120.8, 128.6)
- added ?: , FreqSynth:VIA, F.Cu at (102.8, 104.8)
- added ?: , FreqSynth:VIA, F.Cu at (122.3, 126.8)
- added ?: , FreqSynth:VIA, F.Cu at (123.3, 127.8)
- added ?: , FreqSynth:VIA, F.Cu at (122.3, 124.8)
- added ?: , FreqSynth:VIA, F.Cu at (121.3, 123.8)
- added ?: , FreqSynth:VIA, F.Cu at (123.3, 123.8)
- added ?: , FreqSynth:VIA, F.Cu at (123.3, 125.8)
- added ?: , FreqSynth:VIA, F.Cu at (122.3, 122.8)
- added ?: , FreqSynth:VIA, F.Cu at (121.3, 125.8)
- added ?: , FreqSynth:VIA, F.Cu at (123.3, 121.8)
- added ?: , FreqSynth:VIA, F.Cu at (134.2, 146.0)
- added ?: , FreqSynth:VIA, F.Cu at (102.8, 106.8)
- added ?: , FreqSynth:VIA, F.Cu at (138.2, 147.8)
- added ?: , FreqSynth:VIA, F.Cu at (133.2, 146.0)
- added ?: , FreqSynth:VIA, F.Cu at (135.2, 146.0)
- added ?: , FreqSynth:VIA, F.Cu at (137.2, 146.0)
- added ?: , FreqSynth:VIA, F.Cu at (136.2, 146.0)
- added ?: , FreqSynth:VIA, F.Cu at (133.2, 147.8)
- added ?: , FreqSynth:VIA, F.Cu at (132.2, 147.8)
- added ?: , FreqSynth:VIA, F.Cu at (136.2, 147.8)
- added ?: , FreqSynth:VIA, F.Cu at (134.2, 147.8)
- added ?: , FreqSynth:VIA, F.Cu at (135.2, 147.8)
- added ?: , FreqSynth:VIA, F.Cu at (102.8, 102.8)
- added ?: , FreqSynth:VIA, F.Cu at (137.2, 147.8)
- added ?: , FreqSynth:VIA, F.Cu at (140.0, 146.4)
- added ?: , FreqSynth:VIA, F.Cu at (142.0, 144.4)
- added ?: , FreqSynth:VIA, F.Cu at (139.0, 147.4)
- added ?: , FreqSynth:VIA, F.Cu at (141.0, 145.4)
- added ?: , FreqSynth:VIA, F.Cu at (139.2, 145.0)
- added ?: , FreqSynth:VIA, F.Cu at (141.2, 143.0)
- added ?: , FreqSynth:VIA, F.Cu at (138.2, 146.0)
- added ?: , FreqSynth:VIA, F.Cu at (140.2, 144.0)
- added ?: , FreqSynth:VIA, F.Cu at (122.5, 136.6)
- added ?: , FreqSynth:VIA, F.Cu at (109.2, 107.6)
- added ?: , FreqSynth:VIA, F.Cu at (121.5, 137.6)
- added ?: , FreqSynth:VIA, F.Cu at (120.5, 136.6)
- added ?: , FreqSynth:VIA, F.Cu at (119.5, 137.6)
- added ?: , FreqSynth:VIA, F.Cu at (127.6, 130.4)
- added ?: , FreqSynth:VIA, F.Cu at (126.6, 131.4)
- added ?: , FreqSynth:VIA, F.Cu at (128.6, 129.4)
- added ?: , FreqSynth:VIA, F.Cu at (126.5, 127.8)
- added ?: , FreqSynth:VIA, F.Cu at (127.5, 126.8)
- added ?: , FreqSynth:VIA, F.Cu at (126.5, 123.8)
- added ?: , FreqSynth:VIA, F.Cu at (109.2, 105.6)
- added ?: , FreqSynth:VIA, F.Cu at (126.5, 125.8)
- added ?: , FreqSynth:VIA, F.Cu at (127.5, 124.8)
- added ?: , FreqSynth:VIA, F.Cu at (123.2, 109.4)
- added ?: , FreqSynth:VIA, F.Cu at (124.2, 108.4)
- added ?: , FreqSynth:VIA, F.Cu at (123.2, 107.4)
- added ?: , FreqSynth:VIA, F.Cu at (123.2, 111.4)
- added ?: , FreqSynth:VIA, F.Cu at (124.2, 110.4)
- added ?: , FreqSynth:VIA, F.Cu at (123.2, 113.4)
- added ?: , FreqSynth:VIA, F.Cu at (124.2, 112.4)
- added ?: , FreqSynth:VIA, F.Cu at (140.2, 102.0)
- added ?: , FreqSynth:VIA, F.Cu at (138.6, 148.6)
- added ?: , FreqSynth:VIA, F.Cu at (139.2, 103.0)
- added ?: , FreqSynth:VIA, F.Cu at (141.2, 103.0)
- added ?: , FreqSynth:VIA, F.Cu at (136.2, 102.0)
- added ?: , FreqSynth:VIA, F.Cu at (134.2, 102.0)
- added ?: , FreqSynth:VIA, F.Cu at (137.2, 102.8)
- added ?: , FreqSynth:VIA, F.Cu at (138.2, 102.0)
- added ?: , FreqSynth:VIA, F.Cu at (130.2, 102.0)
- added ?: , FreqSynth:VIA, F.Cu at (129.2, 103.0)
- added ?: , FreqSynth:VIA, F.Cu at (132.2, 102.0)
- added ?: , FreqSynth:VIA, F.Cu at (133.2, 103.0)
- added ?: , FreqSynth:VIA, F.Cu at (104.3, 148.4)
- added ?: , FreqSynth:VIA, F.Cu at (136.6, 148.6)
- added ?: , FreqSynth:VIA, F.Cu at (131.2, 103.0)
- added ?: , FreqSynth:VIA, F.Cu at (128.2, 102.0)
- added ?: , FreqSynth:VIA, F.Cu at (126.2, 102.0)
- added ?: , FreqSynth:VIA, F.Cu at (127.2, 103.0)
- added ?: , FreqSynth:VIA, F.Cu at (116.2, 103.8)
- added ?: , FreqSynth:VIA, F.Cu at (118.2, 101.8)
- added ?: , FreqSynth:VIA, F.Cu at (119.2, 102.8)
- added ?: , FreqSynth:VIA, F.Cu at (116.2, 101.8)
- added ?: , FreqSynth:VIA, F.Cu at (118.2, 103.8)
- added ?: , FreqSynth:VIA, F.Cu at (117.2, 102.8)
- added ?: , FreqSynth:VIA, F.Cu at (134.6, 148.6)
- added ?: , FreqSynth:VIA, F.Cu at (112.2, 101.8)
- added ?: , FreqSynth:VIA, F.Cu at (113.2, 102.8)
- added ?: , FreqSynth:VIA, F.Cu at (112.2, 103.8)
- added ?: , FreqSynth:VIA, F.Cu at (115.2, 102.8)
- added ?: , FreqSynth:VIA, F.Cu at (114.2, 103.8)
- added ?: , FreqSynth:VIA, F.Cu at (114.2, 101.8)
- added ?: , FreqSynth:VIA, F.Cu at (109.2, 102.8)
- added ?: , FreqSynth:VIA, F.Cu at (110.2, 103.8)
- added ?: , FreqSynth:VIA, F.Cu at (111.2, 102.8)
- added ?: , FreqSynth:VIA, F.Cu at (110.2, 101.8)
- added ?: , FreqSynth:VIA, F.Cu at (132.6, 148.6)
- added ?: , FreqSynth:VIA, F.Cu at (106.2, 101.8)
- added ?: , FreqSynth:VIA, F.Cu at (104.2, 101.8)
- added ?: , FreqSynth:VIA, F.Cu at (104.2, 103.8)
- added ?: , FreqSynth:VIA, F.Cu at (108.2, 101.8)
- added ?: , FreqSynth:VIA, F.Cu at (107.2, 102.8)
- added ?: , FreqSynth:VIA, F.Cu at (105.2, 102.8)
- added ?: , FreqSynth:VIA, F.Cu at (106.2, 103.8)
- added ?: , FreqSynth:VIA, F.Cu at (108.2, 103.8)
- added ?: , FreqSynth:VIA, F.Cu at (105.3, 109.0)
- added ?: , FreqSynth:VIA, F.Cu at (103.3, 109.0)
- added ?: , FreqSynth:VIA, F.Cu at (130.6, 148.6)
- added ?: , FreqSynth:VIA, F.Cu at (102.3, 110.0)
- added ?: , FreqSynth:VIA, F.Cu at (103.3, 111.0)
- added ?: , FreqSynth:VIA, F.Cu at (102.3, 112.0)
- added ?: , FreqSynth:VIA, F.Cu at (104.3, 112.0)
- added ?: , FreqSynth:VIA, F.Cu at (106.3, 112.0)
- added ?: , FreqSynth:VIA, F.Cu at (105.3, 111.0)
- added ?: , FreqSynth:VIA, F.Cu at (106.3, 110.0)
- added ?: , FreqSynth:VIA, F.Cu at (104.3, 110.0)
- added ?: , FreqSynth:VIA, F.Cu at (111.3, 109.2)
- added ?: , FreqSynth:VIA, F.Cu at (111.3, 111.2)
- added ?: , FreqSynth:VIA, F.Cu at (147.2, 148.2)
- added ?: , FreqSynth:VIA, F.Cu at (111.3, 113.2)
- added ?: , FreqSynth:VIA, F.Cu at (112.3, 114.2)
- added ?: , FreqSynth:VIA, F.Cu at (114.3, 110.2)
- added ?: , FreqSynth:VIA, F.Cu at (115.3, 111.2)
- added ?: , FreqSynth:VIA, F.Cu at (115.3, 109.2)
- added ?: , FreqSynth:VIA, F.Cu at (113.3, 109.2)
- added ?: , FreqSynth:VIA, F.Cu at (112.3, 112.2)
- added ?: , FreqSynth:VIA, F.Cu at (112.3, 110.2)
- added ?: , FreqSynth:VIA, F.Cu at (113.3, 113.2)
- added ?: , FreqSynth:VIA, F.Cu at (113.3, 111.2)
- added ?: , FreqSynth:VIA, F.Cu at (145.2, 148.2)
- added ?: , FreqSynth:VIA, F.Cu at (114.3, 114.2)
- added ?: , FreqSynth:VIA, F.Cu at (116.3, 114.2)
- added ?: , FreqSynth:VIA, F.Cu at (115.3, 113.2)
- added ?: , FreqSynth:VIA, F.Cu at (116.3, 112.2)
- added ?: , FreqSynth:VIA, F.Cu at (114.3, 112.2)
- added ?: , FreqSynth:VIA, F.Cu at (102.2, 125.4)
- added ?: , FreqSynth:VIA, F.Cu at (102.2, 131.4)
- added ?: , FreqSynth:VIA, F.Cu at (101.2, 130.4)
- added ?: , FreqSynth:VIA, F.Cu at (103.2, 130.4)
- added ?: , FreqSynth:VIA, F.Cu at (105.2, 130.4)
- added ?: , FreqSynth:VIA, F.Cu at (143.2, 148.2)
- added ?: , FreqSynth:VIA, F.Cu at (106.2, 129.4)
- added ?: , FreqSynth:VIA, F.Cu at (104.2, 131.4)
- added ?: , FreqSynth:VIA, F.Cu at (106.2, 131.4)
- added ?: , FreqSynth:VIA, F.Cu at (103.2, 126.4)
- added ?: , FreqSynth:VIA, F.Cu at (103.2, 124.4)
- added ?: , FreqSynth:VIA, F.Cu at (105.2, 126.4)
- added ?: , FreqSynth:VIA, F.Cu at (106.2, 125.4)
- added ?: , FreqSynth:VIA, F.Cu at (105.2, 124.4)
- added ?: , FreqSynth:VIA, F.Cu at (104.2, 125.4)
- added ?: , FreqSynth:VIA, F.Cu at (106.2, 127.4)
- added ?: , FreqSynth:VIA, F.Cu at (141.2, 148.2)
- added ?: , FreqSynth:VIA, F.Cu at (104.2, 129.4)
- added ?: , FreqSynth:VIA, F.Cu at (104.2, 127.4)
- added ?: , FreqSynth:VIA, F.Cu at (105.2, 128.4)
- added ?: , FreqSynth:VIA, F.Cu at (101.2, 136.4)
- added ?: , FreqSynth:VIA, F.Cu at (102.2, 139.2)
- added ?: , FreqSynth:VIA, F.Cu at (101.2, 138.4)
- added ?: , FreqSynth:VIA, F.Cu at (102.2, 137.4)
- added ?: , FreqSynth:VIA, F.Cu at (103.2, 138.4)
- added ?: , FreqSynth:VIA, F.Cu at (103.2, 136.4)
- added ?: , FreqSynth:VIA, F.Cu at (105.2, 134.4)
- added ?: , FreqSynth:VIA, F.Cu at (141.6, 146.6)
- added ?: , FreqSynth:VIA, F.Cu at (104.2, 133.4)
- added ?: , FreqSynth:VIA, F.Cu at (105.2, 132.4)
- added ?: , FreqSynth:VIA, F.Cu at (104.2, 135.4)
- added ?: , FreqSynth:VIA, F.Cu at (106.2, 135.4)
- added ?: , FreqSynth:VIA, F.Cu at (106.2, 133.4)
- added ?: , FreqSynth:VIA, F.Cu at (104.2, 139.2)
- added ?: , FreqSynth:VIA, F.Cu at (104.2, 137.4)
- added ?: , FreqSynth:VIA, F.Cu at (105.2, 138.2)
- added ?: , FreqSynth:VIA, F.Cu at (105.2, 136.4)
- added ?: , FreqSynth:VIA, F.Cu at (106.2, 137.2)
- added ?: , FreqSynth:VIA, F.Cu at (138.2, 142.2)
- added ?: , FreqSynth:VIA, F.Cu at (106.2, 139.4)
- added ?: , FreqSynth:VIA, F.Cu at (103.2, 132.4)
- added ?: , FreqSynth:VIA, F.Cu at (103.2, 134.4)
- added ?: , FreqSynth:VIA, F.Cu at (101.2, 134.4)
- added ?: , FreqSynth:VIA, F.Cu at (102.2, 133.4)
- added ?: , FreqSynth:VIA, F.Cu at (102.2, 135.4)
- added ? (x2): , FreqSynth:VIA, F.Cu at (101.2, 132.4)
- added ?: , FreqSynth:VIA, F.Cu at (102.2, 127.4)
- added ?: , FreqSynth:VIA, F.Cu at (101.2, 128.4)
- added ?: , FreqSynth:VIA, F.Cu at (103.2, 128.4)
- added ?: , FreqSynth:VIA, F.Cu at (103.3, 147.4)
- added ?: , FreqSynth:VIA, F.Cu at (141.2, 141.2)
- added ?: , FreqSynth:VIA, F.Cu at (102.2, 129.4)
- added ?: , FreqSynth:VIA, F.Cu at (111.8, 132.0)
- added ?: , FreqSynth:VIA, F.Cu at (111.8, 134.0)
- added ?: , FreqSynth:VIA, F.Cu at (110.6, 119.8)
- added ?: , FreqSynth:VIA, F.Cu at (115.5, 134.0)
- added ?: , FreqSynth:VIA, F.Cu at (113.5, 134.0)
- added ?: , FreqSynth:VIA, F.Cu at (114.5, 133.0)
- added ?: , FreqSynth:VIA, F.Cu at (115.5, 132.0)
- added ?: , FreqSynth:VIA, F.Cu at (113.5, 132.0)
- added ?: , FreqSynth:VIA, F.Cu at (110.5, 114.2)
- added ?: , FreqSynth:VIA, F.Cu at (140.2, 140.2)
- added ?: , FreqSynth:VIA, F.Cu at (108.5, 114.2)
- added ?: , FreqSynth:VIA, F.Cu at (111.8, 128.0)
- added ?: , FreqSynth:VIA, F.Cu at (111.8, 130.0)
- added ?: , FreqSynth:VIA, F.Cu at (125.2, 124.4)
- added ?: , FreqSynth:VIA, F.Cu at (125.2, 127.4)
- added ?: , FreqSynth:VIA, F.Cu at (125.2, 128.4)
- added ?: , FreqSynth:VIA, F.Cu at (125.2, 126.4)
- added ?: , FreqSynth:VIA, F.Cu at (125.2, 125.4)
- added ?: , FreqSynth:VIA, F.Cu at (125.2, 117.4)
- added ?: , FreqSynth:VIA, F.Cu at (125.2, 116.4)
- added ?: , FreqSynth:VIA, F.Cu at (140.2, 142.2)
- added ?: , FreqSynth:VIA, F.Cu at (125.2, 115.4)
- added ?: , FreqSynth:VIA, F.Cu at (125.2, 133.4)
- added ?: , FreqSynth:VIA, F.Cu at (125.2, 129.4)
- added ?: , FreqSynth:VIA, F.Cu at (125.2, 123.4)
- added ?: , FreqSynth:VIA, F.Cu at (125.2, 121.4)
- added ?: , FreqSynth:VIA, F.Cu at (125.2, 119.4)
- added ?: , FreqSynth:VIA, F.Cu at (125.2, 122.4)
- added ?: , FreqSynth:VIA, F.Cu at (125.2, 120.4)
- added ?: , FreqSynth:VIA, F.Cu at (124.6, 102.2)
- added ?: , FreqSynth:VIA, F.Cu at (124.6, 103.2)
- added ?: , FreqSynth:VIA, F.Cu at (139.2, 143.2)
- added ?: , FreqSynth:VIA, F.Cu at (125.2, 107.4)
- added ?: , FreqSynth:VIA, F.Cu at (125.2, 110.4)
- added ?: , FreqSynth:VIA, F.Cu at (125.2, 111.4)
- added ?: , FreqSynth:VIA, F.Cu at (125.2, 109.4)
- added ?: , FreqSynth:VIA, F.Cu at (125.2, 108.4)
- added ?: , FreqSynth:VIA, F.Cu at (125.2, 143.2)
- added ?: , FreqSynth:VIA, F.Cu at (125.2, 136.4)
- added ?: , FreqSynth:VIA, F.Cu at (125.2, 137.4)
- added ?: , FreqSynth:VIA, F.Cu at (125.2, 138.4)
- added ?: , FreqSynth:VIA, F.Cu at (125.2, 140.4)
- added ?: , FreqSynth:VIA, F.Cu at (139.2, 141.2)
- added ?: , FreqSynth:VIA, F.Cu at (125.2, 135.4)
- added ?: , FreqSynth:VIA, F.Cu at (125.2, 146.4)
- added ?: , FreqSynth:VIA, F.Cu at (148.6, 127.2)
- added ?: , FreqSynth:VIA, F.Cu at (148.6, 147.6)
- added ?: , FreqSynth:VIA, F.Cu at (148.6, 148.6)
- added ?: , FreqSynth:VIA, F.Cu at (147.8, 138.8)
- added ?: , FreqSynth:VIA, F.Cu at (148.6, 137.2)
- added ?: , FreqSynth:VIA, F.Cu at (148.6, 138.2)
- added ?: , FreqSynth:VIA, F.Cu at (148.6, 135.2)
- added ?: , FreqSynth:VIA, F.Cu at (148.6, 136.2)
- added ?: , FreqSynth:VIA, F.Cu at (137.2, 143.2)
- added ?: , FreqSynth:VIA, F.Cu at (148.6, 133.2)
- added ?: , FreqSynth:VIA, F.Cu at (148.6, 134.2)
- added ?: , FreqSynth:VIA, F.Cu at (148.6, 131.2)
- added ?: , FreqSynth:VIA, F.Cu at (148.6, 129.2)
- added ?: , FreqSynth:VIA, F.Cu at (148.6, 130.2)
- added ?: , FreqSynth:VIA, F.Cu at (148.6, 128.2)
- added ?: , FreqSynth:VIA, F.Cu at (148.6, 132.2)
- added ?: , FreqSynth:VIA, F.Cu at (148.6, 118.2)
- added ?: , FreqSynth:VIA, F.Cu at (148.6, 117.2)
- added ?: , FreqSynth:VIA, F.Cu at (148.6, 111.2)
- added ?: , FreqSynth:VIA, F.Cu at (137.2, 145.2)
- added ?: , FreqSynth:VIA, F.Cu at (148.6, 114.2)
- added ?: , FreqSynth:VIA, F.Cu at (148.6, 115.2)
- added ?: , FreqSynth:VIA, F.Cu at (148.6, 112.2)
- added ?: , FreqSynth:VIA, F.Cu at (148.6, 116.2)
- added ?: , FreqSynth:VIA, F.Cu at (148.6, 113.2)
- added ?: , FreqSynth:VIA, F.Cu at (148.6, 102.2)
- added ?: , FreqSynth:VIA, F.Cu at (101.2, 116.4)
- added ?: , FreqSynth:VIA, F.Cu at (101.2, 118.4)
- added ?: , FreqSynth:VIA, F.Cu at (101.2, 117.4)
- added ?: , FreqSynth:VIA, F.Cu at (101.2, 114.4)
- added ?: , FreqSynth:VIA, F.Cu at (136.2, 144.2)
- added ?: , FreqSynth:VIA, F.Cu at (101.2, 115.4)
- added ?: , FreqSynth:VIA, F.Cu at (101.2, 113.4)
- added ?: , FreqSynth:VIA, F.Cu at (101.2, 112.4)
- added ?: , FreqSynth:VIA, F.Cu at (101.2, 111.4)
- added ?: , FreqSynth:VIA, F.Cu at (101.2, 109.4)
- added ?: , FreqSynth:VIA, F.Cu at (101.2, 110.4)
- added ?: , FreqSynth:VIA, F.Cu at (101.2, 108.4)
- added ?: , FreqSynth:VIA, F.Cu at (101.2, 104.4)
- added ?: , FreqSynth:VIA, F.Cu at (101.2, 103.4)
- added ?: , FreqSynth:VIA, F.Cu at (101.2, 102.4)
- added ?: , FreqSynth:VIA, F.Cu at (138.2, 144.2)
- added ?: , FreqSynth:VIA, F.Cu at (101.2, 107.4)
- added ?: , FreqSynth:VIA, F.Cu at (101.2, 106.4)
- added ?: , FreqSynth:VIA, F.Cu at (101.2, 105.4)
- added ?: , FreqSynth:VIA, F.Cu at (101.2, 121.4)
- added ?: , FreqSynth:VIA, F.Cu at (101.2, 120.4)
- added ?: , FreqSynth:VIA, F.Cu at (101.2, 122.4)
- added ?: , FreqSynth:VIA, F.Cu at (101.2, 119.4)
- added ?: , FreqSynth:VIA, F.Cu at (101.2, 125.4)
- added ?: , FreqSynth:VIA, F.Cu at (101.2, 123.4)
- added ?: , FreqSynth:VIA, F.Cu at (101.2, 124.4)
- added ?: , FreqSynth:VIA, F.Cu at (139.6, 130.6)
- added ?: , FreqSynth:VIA, F.Cu at (101.2, 127.4)
- added ?: , FreqSynth:VIA, F.Cu at (101.2, 126.4)
- added ?: , FreqSynth:VIA, F.Cu at (101.2, 145.4)
- added ?: , FreqSynth:VIA, F.Cu at (101.2, 148.4)
- added ?: , FreqSynth:VIA, F.Cu at (101.2, 143.4)
- added ?: , FreqSynth:VIA, F.Cu at (101.2, 144.4)
- added ?: , FreqSynth:VIA, F.Cu at (101.2, 147.4)
- added ?: , FreqSynth:VIA, F.Cu at (101.2, 146.4)
- added ?: , FreqSynth:VIA, F.Cu at (101.2, 140.4)
- added ?: , FreqSynth:VIA, F.Cu at (101.2, 141.4)
- added ?: , FreqSynth:VIA, F.Cu at (102.3, 148.4)
- added ?: , FreqSynth:VIA, F.Cu at (140.7, 129.6)
- added ?: , FreqSynth:VIA, F.Cu at (101.2, 149.4)
- added ?: , FreqSynth:VIA, F.Cu at (101.2, 142.4)
- added ?: , FreqSynth:VIA, F.Cu at (101.2, 129.4)
- added ?: , FreqSynth:VIA, F.Cu at (101.2, 131.4)
- added ?: , FreqSynth:VIA, F.Cu at (101.2, 133.4)
- added ?: , FreqSynth:VIA, F.Cu at (101.2, 135.4)
- added ?: , FreqSynth:VIA, F.Cu at (101.2, 139.4)
- added ?: , FreqSynth:VIA, F.Cu at (101.2, 137.4)
- added ?: , FreqSynth:VIA, F.Cu at (138.2, 149.4)
- added ?: , FreqSynth:VIA, F.Cu at (138.4, 129.8)
- added ?: , FreqSynth:VIA, F.Cu at (137.2, 149.4)
- added ?: , FreqSynth:VIA, F.Cu at (135.2, 149.4)
- added ?: , FreqSynth:VIA, F.Cu at (133.2, 149.4)
- added ?: , FreqSynth:VIA, F.Cu at (134.2, 149.4)
- added ?: , FreqSynth:VIA, F.Cu at (132.2, 149.4)
- added ?: , FreqSynth:VIA, F.Cu at (136.2, 149.4)
- added ?: , FreqSynth:VIA, F.Cu at (148.2, 149.4)
- added ?: , FreqSynth:VIA, F.Cu at (145.2, 149.4)
- added ?: , FreqSynth:VIA, F.Cu at (144.2, 149.4)
- added ?: , FreqSynth:VIA, F.Cu at (147.2, 149.4)
- added ?: , FreqSynth:VIA, F.Cu at (140.7, 127.5)
- added ?: , FreqSynth:VIA, F.Cu at (146.2, 149.4)
- added ?: , FreqSynth:VIA, F.Cu at (140.2, 149.4)
- added ?: , FreqSynth:VIA, F.Cu at (139.2, 149.4)
- added ?: , FreqSynth:VIA, F.Cu at (141.2, 149.4)
- added ?: , FreqSynth:VIA, F.Cu at (142.2, 149.4)
- added ?: , FreqSynth:VIA, F.Cu at (143.2, 149.4)
- added ?: , FreqSynth:VIA, F.Cu at (131.2, 149.4)
- added ?: , FreqSynth:VIA, F.Cu at (128.2, 149.4)
- added ?: , FreqSynth:VIA, F.Cu at (130.2, 149.4)
- added ?: , FreqSynth:VIA, F.Cu at (129.2, 149.4)
- added ?: , FreqSynth:VIA, F.Cu at (139.6, 128.6)
- added ?: , FreqSynth:VIA, F.Cu at (126.2, 149.4)
- added ?: , FreqSynth:VIA, F.Cu at (127.2, 149.4)
- added ?: , FreqSynth:VIA, F.Cu at (125.2, 149.4)
- added ?: , FreqSynth:VIA, F.Cu at (124.2, 149.4)
- added ?: , FreqSynth:VIA, F.Cu at (122.2, 149.4)
- added ?: , FreqSynth:VIA, F.Cu at (123.2, 149.4)
- added ?: , FreqSynth:VIA, F.Cu at (107.2, 149.4)
- added ?: , FreqSynth:VIA, F.Cu at (108.2, 149.4)
- added ?: , FreqSynth:VIA, F.Cu at (106.2, 149.4)
- added ?: , FreqSynth:VIA, F.Cu at (113.2, 149.4)
- added ?: , FreqSynth:VIA, F.Cu at (143.9, 136.8)
- added ?: , FreqSynth:VIA, F.Cu at (114.2, 149.4)
- added ?: , FreqSynth:VIA, F.Cu at (110.2, 149.4)
- added ?: , FreqSynth:VIA, F.Cu at (111.2, 149.4)
- added ?: , FreqSynth:VIA, F.Cu at (112.2, 149.4)
- added ?: , FreqSynth:VIA, F.Cu at (109.2, 149.4)
- added ?: , FreqSynth:VIA, F.Cu at (105.2, 149.4)
- added ?: , FreqSynth:VIA, F.Cu at (102.2, 149.4)
- added ?: , FreqSynth:VIA, F.Cu at (103.2, 149.4)
- added ?: , FreqSynth:VIA, F.Cu at (104.2, 149.4)
- added ?: , FreqSynth:VIA, F.Cu at (115.2, 149.4)
- added ?: , FreqSynth:VIA, F.Cu at (145.9, 136.8)
- added ?: , FreqSynth:VIA, F.Cu at (116.2, 149.4)
- added ?: , FreqSynth:VIA, F.Cu at (117.2, 149.4)
- added ?: , FreqSynth:VIA, F.Cu at (119.2, 149.4)
- added ?: , FreqSynth:VIA, F.Cu at (118.2, 149.4)
- added ?: , FreqSynth:VIA, F.Cu at (120.2, 149.4)
- added ?: , FreqSynth:VIA, F.Cu at (121.2, 149.4)
- added ?: , FreqSynth:VIA, F.Cu at (108.6, 101.2)
- added ?: , FreqSynth:VIA, F.Cu at (107.6, 101.2)
- added ?: , FreqSynth:VIA, F.Cu at (110.6, 101.2)
- added ?: , FreqSynth:VIA, F.Cu at (109.6, 101.2)
- added ?: , FreqSynth:VIA, F.Cu at (146.9, 137.8)
- added ?: , FreqSynth:VIA, F.Cu at (111.6, 101.2)
- added ?: , FreqSynth:VIA, F.Cu at (112.6, 101.2)
- added ?: , FreqSynth:VIA, F.Cu at (115.6, 101.2)
- added ?: , FreqSynth:VIA, F.Cu at (114.6, 101.2)
- added ?: , FreqSynth:VIA, F.Cu at (113.6, 101.2)
- added ?: , FreqSynth:VIA, F.Cu at (117.6, 101.2)
- added ?: , FreqSynth:VIA, F.Cu at (116.6, 101.2)
- added ?: , FreqSynth:VIA, F.Cu at (106.6, 101.2)
- added ?: , FreqSynth:VIA, F.Cu at (104.6, 101.2)
- added ?: , FreqSynth:VIA, F.Cu at (105.6, 101.2)
- added ?: , FreqSynth:VIA, F.Cu at (144.9, 135.8)
- added ?: , FreqSynth:VIA, F.Cu at (101.6, 101.2)
- added ?: , FreqSynth:VIA, F.Cu at (102.6, 101.2)
- added ?: , FreqSynth:VIA, F.Cu at (103.6, 101.2)
- added ?: , FreqSynth:VIA, F.Cu at (138.6, 101.2)
- added ?: , FreqSynth:VIA, F.Cu at (137.6, 101.2)
- added ?: , FreqSynth:VIA, F.Cu at (140.6, 101.2)
- added ?: , FreqSynth:VIA, F.Cu at (139.6, 101.2)
- added ?: , FreqSynth:VIA, F.Cu at (141.6, 101.2)
- added ?: , FreqSynth:VIA, F.Cu at (142.6, 101.2)
- added ?: , FreqSynth:VIA, F.Cu at (145.6, 101.2)
- added ?: , FreqSynth:VIA, F.Cu at (146.9, 135.8)
- added ?: , FreqSynth:VIA, F.Cu at (144.6, 101.2)
- added ?: , FreqSynth:VIA, F.Cu at (143.6, 101.2)
- added ?: , FreqSynth:VIA, F.Cu at (147.6, 101.2)
- added ?: , FreqSynth:VIA, F.Cu at (146.6, 101.2)
- added ?: , FreqSynth:VIA, F.Cu at (148.6, 101.2)
- added ?: , FreqSynth:VIA, F.Cu at (136.6, 101.2)
- added ?: , FreqSynth:VIA, F.Cu at (134.6, 101.2)
- added ?: , FreqSynth:VIA, F.Cu at (135.6, 101.2)
- added ?: , FreqSynth:VIA, F.Cu at (128.6, 101.2)
- added ?: , FreqSynth:VIA, F.Cu at (130.6, 101.2)
- added ?: , FreqSynth:VIA, F.Cu at (144.9, 137.8)
- added ?: , FreqSynth:VIA, F.Cu at (131.6, 101.2)
- added ?: , FreqSynth:VIA, F.Cu at (132.6, 101.2)
- added ?: , FreqSynth:VIA, F.Cu at (133.6, 101.2)
- added ?: , FreqSynth:VIA, F.Cu at (129.6, 101.2)
- added ?: , FreqSynth:VIA, F.Cu at (125.6, 101.2)
- added ?: , FreqSynth:VIA, F.Cu at (124.6, 101.2)
- added ?: , FreqSynth:VIA, F.Cu at (126.6, 101.2)
- added ?: , FreqSynth:VIA, F.Cu at (127.6, 101.2)
- added ?: , FreqSynth:VIA, F.Cu at (123.6, 101.2)
- added ?: , FreqSynth:VIA, F.Cu at (118.6, 101.2)
- added ?: , FreqSynth:VIA, F.Cu at (108.2, 143.8)
- added ?: , FreqSynth:VIA, F.Cu at (145.9, 130.8)
- added ?: , FreqSynth:VIA, F.Cu at (120.6, 101.2)
- added ?: , FreqSynth:VIA, F.Cu at (119.6, 101.2)
- added ?: , FreqSynth:VIA, F.Cu at (121.6, 101.2)
- added ?: , FreqSynth:VIA, F.Cu at (122.6, 101.2)
- added ?: , FreqSynth:VIA, F.Cu at (142.0, 108.2)
- added ?: , FreqSynth:VIA, F.Cu at (147.0, 126.4)
- added ?: , FreqSynth:VIA, F.Cu at (147.0, 104.4)
- added ?: , FreqSynth:VIA, F.Cu at (147.0, 121.6)
- added ?: , FreqSynth:VIA, F.Cu at (147.0, 120.6)
- added ?: , FreqSynth:VIA, F.Cu at (147.0, 105.4)
- added ?: , FreqSynth:VIA, F.Cu at (144.9, 131.8)
- added ?: , FreqSynth:VIA, F.Cu at (147.0, 108.2)
- added ?: , FreqSynth:VIA, F.Cu at (147.0, 124.4)
- added ?: , FreqSynth:VIA, F.Cu at (147.0, 109.2)
- added ?: , FreqSynth:VIA, F.Cu at (147.0, 110.2)
- added ?: , FreqSynth:VIA, F.Cu at (147.0, 125.4)
- added ?: , FreqSynth:VIA, F.Cu at (147.0, 119.6)
- added ?: , FreqSynth:VIA, F.Cu at (147.0, 103.4)
- added ?: , FreqSynth:VIA, F.Cu at (146.9, 131.8)
- added ?: , FreqSynth:VIA, F.Cu at (143.9, 130.8)
- added ?: , FreqSynth:VIA, F.Cu at (145.9, 134.8)
- added ?: , FreqSynth:VIA, F.Cu at (146.9, 133.8)
- added ?: , FreqSynth:VIA, F.Cu at (144.9, 133.8)
- added ?: , FreqSynth:VIA, F.Cu at (145.9, 132.8)
- added ?: , FreqSynth:VIA, F.Cu at (142.9, 135.8)
- added ?: , FreqSynth:VIA, F.Cu at (142.9, 137.8)
- added ?: , FreqSynth:VIA, F.Cu at (108.2, 145.8)
- added ?: , FreqSynth:VIA, F.Cu at (146.9, 129.8)
- added ?: , FreqSynth:VIA, F.Cu at (144.9, 129.8)
- added ?: , FreqSynth:VIA, F.Cu at (144.9, 127.8)
- added ?: , FreqSynth:VIA, F.Cu at (146.9, 127.8)
- added ?: , FreqSynth:VIA, F.Cu at (145.9, 128.8)
- added ?: , FreqSynth:VIA, F.Cu at (142.9, 129.8)
- added ?: , FreqSynth:VIA, F.Cu at (142.9, 127.8)
- added ?: , FreqSynth:VIA, F.Cu at (143.9, 128.8)
- added ?: , FreqSynth:VIA, F.Cu at (141.9, 119.2)
- added ?: , FreqSynth:VIA, F.Cu at (141.9, 121.2)
- added ?: , FreqSynth:VIA, F.Cu at (108.2, 147.8)
- added ?: , FreqSynth:VIA, F.Cu at (139.8, 123.0)
- added ?: , FreqSynth:VIA, F.Cu at (139.8, 121.0)
- added ?: , FreqSynth:VIA, F.Cu at (139.8, 119.0)
- added ?: , FreqSynth:VIA, F.Cu at (139.8, 117.0)
- added ?: , FreqSynth:VIA, F.Cu at (139.8, 115.0)
- added ?: , FreqSynth:VIA, F.Cu at (144.9, 118.2)
- added ?: , FreqSynth:VIA, F.Cu at (145.9, 117.2)
- added ?: , FreqSynth:VIA, F.Cu at (146.9, 118.2)
- added ?: , FreqSynth:VIA, F.Cu at (146.9, 114.2)
- added ?: , FreqSynth:VIA, F.Cu at (144.9, 116.2)
- added ?: , FreqSynth:VIA, F.Cu at (108.2, 141.8)
- added ?: , FreqSynth:VIA, F.Cu at (146.9, 116.2)
- added ?: , FreqSynth:VIA, F.Cu at (145.9, 115.2)
- added ?: , FreqSynth:VIA, F.Cu at (144.9, 114.2)
- added ?: , FreqSynth:VIA, F.Cu at (143.9, 113.2)
- added ?: , FreqSynth:VIA, F.Cu at (142.9, 112.2)
- added ?: , FreqSynth:VIA, F.Cu at (143.9, 111.2)
- added ?: , FreqSynth:VIA, F.Cu at (142.9, 114.2)
- added ?: , FreqSynth:VIA, F.Cu at (142.9, 118.2)
- added ?: , FreqSynth:VIA, F.Cu at (143.9, 117.2)
- added ?: , FreqSynth:VIA, F.Cu at (142.9, 116.2)
- added ?: , FreqSynth:VIA, F.Cu at (115.8, 139.8)
- added ?: , FreqSynth:VIA, F.Cu at (143.9, 115.2)
- added ?: , FreqSynth:VIA, F.Cu at (145.9, 111.2)
- added ?: , FreqSynth:VIA, F.Cu at (146.9, 112.2)
- added ?: , FreqSynth:VIA, F.Cu at (145.9, 113.2)
- added ?: , FreqSynth:VIA, F.Cu at (144.9, 112.2)
- added ?: , FreqSynth:VIA, F.Cu at (141.9, 115.2)
- added ?: , FreqSynth:VIA, F.Cu at (141.9, 113.2)
- added ?: , FreqSynth:VIA, F.Cu at (141.9, 111.2)
- added ?: , FreqSynth:VIA, F.Cu at (141.9, 117.2)
- added ?: , FreqSynth:VIA, F.Cu at (127.2, 120.2)
- added G***: LOGO, FreqSynth:Logo_silk_polarity_center_5x1.4mm, B.Cu at (103.0, 106.8)
- added G***: LOGO, FreqSynth:Logo_silk_OSHW_6x6mm, B.Cu at (122.0, 142.0)
- moved ? 31.0 mm to (126.4, 115.0)
- moved ? 0.27 mm to (138.8, 110.5)
- moved ? 0.20 mm to (131.6, 129.0)
- moved ? 0.20 mm to (132.6, 129.0)
- moved ? 0.05 mm to (132.8, 125.2)
- moved ? 0.05 mm to (134.1, 125.2)
Routing:
- net /SCK: track 1.20 -> 79.1 mm, vias 1 -> 4
- net /MOSI: track 0.70 -> 74.4 mm, vias 1 -> 3
- net /MCU/ADC1: track 0.76 -> 48.4 mm, vias 1 -> 2
- net /MCU/VCC_D: track 10.9 -> 56.1 mm, vias 2 -> 3
- net /Amplifier/PWDN: track 1.00 -> 46.0 mm, vias 1 -> 2
- net /FILT2: track 0.90 -> 41.7 mm, vias 1 -> 3
- net /FILT1: track 1.00 -> 39.4 mm, vias 1 -> 3
- net /FILT4: track 1.00 -> 34.3 mm, vias 1 -> 3
- net /FILT3: track 0.90 -> 33.7 mm, vias 1 -> 3
- net /3v3: track 26.9 -> 59.3 mm, vias 2 -> 10
- net /MISO: track 0.89 -> 28.0 mm, vias 1 -> 2
- net /MCU/CS_PLL: track 2.10 -> 23.2 mm
- net /Amplifier/ATTEN_CS: track 18.7 -> 38.2 mm, vias 1 -> 2
- net /MCU/CE_PLL: track 1.60 -> 20.3 mm
- net Earth: track 127.9 -> 143.1 mm, vias 24 -> 40
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Other:
- outline, holes or cut-outs redrawn
